Commit message: exam_robot

File: src/my_robot_controller/urdf/simple_robot.urdf (robot description, URDF)
Before this commit: robot simple_robot, 6 links, 5 joints
Links:
- removed link imu_link
- added link led_back_left_link; visual sphere radius=0.01
- added link led_back_right_link; visual sphere radius=0.01
- added link led_front_left_link; visual sphere radius=0.01
- added link led_front_right_link; visual sphere radius=0.01
- added link wheel_left_back_link; visual cylinder length=0.05 radius=0.1
- added link wheel_right_back_link; visual cylinder length=0.05 radius=0.1
- link wheel_left_link: mass 0.5 -> None; geometry visual cylinder length=0.05 radius=0.1
- link wheel_right_link: mass 0.5 -> None; geometry visual cylinder length=0.05 radius=0.1
Joints:
- removed joint base_to_imu
- added joint base_to_led_back_left: type fixed, parent base_link, child led_back_left_link, origin xyz=-0.2 0.12 0.05 rpy=0 0 0
- added joint base_to_led_back_right: type fixed, parent base_link, child led_back_right_link, origin xyz=-0.2 -0.12 0.05 rpy=0 0 0
- added joint base_to_led_front_left: type fixed, parent base_link, child led_front_left_link, origin xyz=0.2 0.12 0.05 rpy=0 0 0
- added joint base_to_led_front_right: type fixed, parent base_link, child led_front_right_link, origin xyz=0.2 -0.12 0.05 rpy=0 0 0
- added joint base_to_left_back_wheel: type continuous, parent base_link, child wheel_left_back_link, origin xyz=-0.15 0.175 0 rpy=1.5708 0 0, axis 0 0 1
- added joint base_to_right_back_wheel: type continuous, parent base_link, child wheel_right_back_link, origin xyz=-0.15 -0.175 0 rpy=1.5708 0 0, axis 0 0 1
- joint base_to_left_wheel: origin xyz=0 0.175 0 rpy=1.5708 0 0 -> xyz=0.15 0.175 0 rpy=1.5708 0 0
- joint base_to_right_wheel: origin xyz=0 -0.175 0 rpy=1.5708 0 0 -> xyz=0.15 -0.175 0 rpy=1.5708 0 0
