Commit message: Контрольная изменения

File: src/exam_robot/urdf/exam_robot.urdf (robot description, URDF)
Before this commit: robot exam_robot, 4 links, 3 joints
Joints:
- joint left_wheel_joint: axis 0 1 0 -> (none); origin xyz=0 0.17 0 rpy=0 0 0 -> xyz=0 0.17 -0.06 rpy=1.5708 0 0; type continuous -> fixed
- joint right_wheel_joint: axis 0 1 0 -> (none); origin xyz=0 -0.17 0 rpy=0 0 0 -> xyz=0 -0.17 -0.06 rpy=1.5708 0 0; type continuous -> fixed
